File: simulations/simulations.kicad_sch (KiCad schematic)
At the start: 41 parts, among them Q1 NPN, Q2 NPN, Q3 NPN, Q4 NPN, U1 ${SIM.PARAMS}, U2 ${SIM.PARAMS}, U3 ${SIM.PARAMS}, U4 ${SIM.PARAMS}, U5 ${SIM.PARAMS}, U6 ${SIM.PARAMS}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

Commit message: Added simulations
Parts:
- added Q5, Q6: NPN, symbol Simulation_SPICE:NPN
- added R24, R25: 10k, symbol Device:R
- added R26: 220, symbol Device:R
- added R27: 100k, symbol Device:R
- added R28, R29: 470, symbol Device:R
- added R30, R31: 33k, symbol Device:R
- added R32, R33: 25k, symbol Device:R
- added U10: ${SIM.PARAMS}, symbol Simulation_SPICE:OPAMP
- R1, R2: value 100k -> 10k
- R20: value 47k -> 20k
- R22: value 50k -> 47k
- R23: value 20k -> 10k
- R3: value 47k -> 58k
Connections:
- net +12V: now also R24.2, R25.2, U10.3 (V+); no longer R1.1
- net -12V: now also R32.2, R33.1, U10.4 (V-)
- net GND: now also U3.1 (+), R28.2, R29.2, R31.2; no longer R2.2
- net RAMP_UP: now also R1.1
- net TRIANGLE: now also R27.2
- net RAMP_REF: now reaches R22.1, R23.1, U9.1 (+)
- net REF_V: no longer names the net of U3.2 (-)
- net REF_V: now also R1.2, R2.1; no longer U3.5
- removed net VREF: R1.2, R2.1, U3.1 (+)
- new net: Q6.1 (C), R25.1, R31.1, U10.1 (+)
- new net: Q5.1 (C), R24.1, R30.2, U10.2 (-)
- new net: Q5.2 (B), R27.1, R28.1
- new net: Q5.3 (E), R26.2, R33.2
- new net: Q6.3 (E), R26.1, R32.1
- new net: Q6.2 (B), R29.1
- new net RAMP_DOWN: R2.2, U3.5
- new net SIN: R30.1, U10.5
Other:
- moved on the sheet: Q4, R15, R16, R17, R18, R19, R20, R21, R22, R23, U7, U8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

Commit message: VCA v. 2.0
Changed lines of the file:
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@@
 		(on_board yes)
 		(dnp no)
-		(fields_autoplaced yes)
 		(property "Reference" "R8"
-			(at 177.8 48.26 90)
+			(at 180.594 57.404 90)
 			(effects
 				(font
@@
 		)
 		(property "Value" "47k"
-			(at 177.8 50.8 90)
+			(at 176.022 58.166 90)
 			(effects
 				(font
