File: linear-vintage-vca/board_front.kicad_pcb (KiCad board)
At the start: 2 copper layers, 30 x 128.5 mm, 17 parts

Commit message: Front panel and output gain fix.
Parts:
- added REF**: Panel Mount Hole, SynthUX_Components:Panel Mount Hole, F.Cu at (111.0, 165.5)
- added REF**: Panel Mount Hole, SynthUX_Components:Panel Mount Hole, F.Cu at (111.0, 43.0)
