File: simulations/exponential-vca/exponential-vca.kicad_sch (KiCad schematic)
At the start: 21 parts, among them Q1 PNP, Q2 PNP, Q3 PNP, Q4 NPN, U1 ${SIM.PARAMS}, U4 ${SIM.PARAMS}

Commit message: E24 series components selected for 0-5V VC and ~<500 uA output.
Parts:
- removed Q4: NPN, symbol Simulation_SPICE:NPN
- added U2: ${SIM.PARAMS}, symbol Simulation_SPICE:OPAMP
- R1: value 6.8k -> 18k
- R2: value 2Meg -> 2.0Meg
- R3: value 2.4k -> 2.2k
- R9: value 2k -> 20k
Connections:
- net +12V: now also U2.3 (V+)
- net -12V: now also U2.4 (V-)
- net CV: now also U2.1 (+); no longer R4.1
- new net: R4.1, U2.2 (-), U2.5
