File: exp-vintage-vca/exp-vintage-vca.kicad_pcb (KiCad board)
At the start: 2 copper layers, 170 x 110 mm, 83 parts, among them J1 AudioJack2, J10 Conn_01x10_Socket, J11 Conn_01x04_Pin, J12 Conn_01x04_Socket, J13 AudioJack2, J14 AudioJack2, J15 Conn_02x08_Odd_Even, J2 AudioJack2, J3 AudioJack2, J4 AudioJack2, J5 AudioJack2, J6 AudioJack2, J7 Conn_01x06_Pin, J8 Conn_01x06_Pin, J9 Conn_01x10_Socket, U1 TL074, U3 LM13700, U4 TL074

Commit message: Exponential VCA ver. 1.2
Parts:
- removed JP1: SolderJumper_2_Open, Jumper:SolderJumper-2_P1.3mm_Open_RoundedPad1.0x1.5mm
- removed TP1, TP2, TP3, TP4: TestPoint, TestPoint:TestPoint_Loop_D1.80mm_Drill1.0mm_Beaded
- added D3: SS14, Diode_SMD:D_SMA, F.Cu at (51.3, 51.8)
- added D5: SS14, Diode_SMD:D_SMA, F.Cu at (53.1, 58.2)
- added FB1: FerriteBead_Small, linear_vintage_vca:Ferrite_Bead_5mm_3.5mm_Horizontal, F.Cu at (38.4, 51.8)
- added FB2: FerriteBead_Small, linear_vintage_vca:Ferrite_Bead_5mm_3.5mm_Horizontal, F.Cu at (43.4, 55.9)
- added R24: 10K, Resistor_SMD:R_0603_1608Metric_Pad0.98x0.95mm_HandSolder, F.Cu at (43.9, 129.3)
- added R35: 10K, Resistor_SMD:R_0603_1608Metric_Pad0.98x0.95mm_HandSolder, F.Cu at (60.6, 97.5)
- added RV10: 20K, Potentiometer_THT:Potentiometer_Bourns_3296W_Vertical, B.Cu at (62.8, 72.3)
- added RV9: 20k, Potentiometer_THT:Potentiometer_Bourns_3296W_Vertical, B.Cu at (38.7, 63.1)
- C11, C12: footprint Capacitor_THT:CP_Radial_D10.0mm_P2.50mm_P5.00mm -> Capacitor_THT:CP_Radial_D5.0mm_P2.50mm
- D1, D2: footprint Diode_SMD:D_0805_2012Metric_Pad1.15x1.40mm_HandSolder -> Diode_SMD:D_SOD-123
- J15: footprint Connector_IDC:IDC-Header_2x08_P2.54mm_Vertical -> Connector_IDC:IDC-Header_2x05_P2.54mm_Vertical
- R10, R13, R14, R18, R21, R22, R29, R3, R4, R5, R6, R7, R8, R9: footprint Resistor_SMD:R_0805_2012Metric_Pad1.20x1.40mm_HandSolder -> Resistor_SMD:R_0603_1608Metric_Pad0.98x0.95mm_HandSolder
- R11, R12, R15, R16: value 620R -> 680R; footprint Resistor_SMD:R_0805_2012Metric_Pad1.20x1.40mm_HandSolder -> Resistor_SMD:R_0603_1608Metric_Pad0.98x0.95mm_HandSolder
- R17, R23: value 330k -> 330K; footprint Resistor_SMD:R_0805_2012Metric_Pad1.20x1.40mm_HandSolder -> Resistor_SMD:R_0603_1608Metric_Pad0.98x0.95mm_HandSolder
- R19, R20: value 20k -> 10K; footprint Resistor_SMD:R_0805_2012Metric_Pad1.20x1.40mm_HandSolder -> Resistor_SMD:R_0603_1608Metric_Pad0.98x0.95mm_HandSolder
- R25, R31: value 330 -> 10; footprint Resistor_SMD:R_0805_2012Metric_Pad1.20x1.40mm_HandSolder -> Resistor_SMD:R_0603_1608Metric_Pad0.98x0.95mm_HandSolder
- R26, R32: value 1Meg -> 2Meg; footprint Resistor_SMD:R_0805_2012Metric_Pad1.20x1.40mm_HandSolder -> Resistor_SMD:R_0603_1608Metric_Pad0.98x0.95mm_HandSolder
- R27, R33: value 22k -> 10K; footprint Resistor_SMD:R_0805_2012Metric_Pad1.20x1.40mm_HandSolder -> Resistor_SMD:R_0603_1608Metric_Pad0.98x0.95mm_HandSolder
- R28, R34: value 6k8 -> 20K; footprint Resistor_SMD:R_0805_2012Metric_Pad1.20x1.40mm_HandSolder -> Resistor_SMD:R_0603_1608Metric_Pad0.98x0.95mm_HandSolder
- RV5, RV6: footprint Potentiometer_THT:Potentiometer_Runtron_RM-065_Vertical -> Potentiometer_THT:Potentiometer_Bourns_3296W_Vertical
- RV7, RV8: value 10k -> 20K; footprint Potentiometer_THT:Potentiometer_Runtron_RM-065_Vertical -> Potentiometer_THT:Potentiometer_Bourns_3296W_Vertical
- U1, U4: footprint Package_SO:SOIC-14_3.9x8.7mm_P1.27mm -> linear_vintage_vca:SOT-23-THIN-14_2x4.2mm_P0.5mm
- U2, U5: value ~ -> BC857BS
- moved RV6 69.1 mm to (62.8, 77.8), turned to 0 degrees
- moved R31 61.5 mm to (61.7, 80.5), turned to 0 degrees
- moved R32 48.4 mm to (42.7, 103.1)
- moved RV8 42.4 mm to (62.8, 83.3), turned to 0 degrees
- moved R18 35.5 mm to (61.7, 104.9), turned to -90 degrees
- moved U5 35.0 mm to (49.0, 113.3)
- moved C4 33.2 mm to (43.4, 106.9), turned to 90 degrees
- moved R33 32.9 mm to (53.0, 115.6), turned to 0 degrees
- moved R29 32.2 mm to (53.5, 111.8), turned to 180 degrees
- moved U4 32.2 mm to (49.0, 108.0)
- moved C13 32.0 mm to (55.0, 108.3)
- moved C14 31.4 mm to (43.7, 112.0), turned to 0 degrees
- moved C2 31.2 mm to (56.6, 104.9)
- moved D2 31.2 mm to (59.2, 104.7)
- moved R14 31.0 mm to (54.8, 105.0)
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Connections:
- C14 pad 1: Net-(U4B-+) -> Net-(U4B--)
- C3 pad 1: Net-(U1D-+) -> Net-(U1D--)
- J1 pad TN: CV_A -> GND_A
- J11 pad 1: CV_A -> GND_A
- J12 pad 1: Net-(J12-Pin_1) -> GND
- J15 pad 1: -12V -> Net-(D5-K)
- J15 pad 10: +12V -> Net-(D3-A)
- J15 pad 2: -12V -> Net-(D5-K)
- J15 pad 9: +12V -> Net-(D3-A)
- J3 pad TN: CV_A -> GND_A
- R10 pad 2: Net-(U3A--) -> Net-(R10-Pad2)
- R26 pad 1: Net-(U1D-+) -> Net-(U1D--)
- R27 pad 1: Net-(U2A-E) -> Net-(U2A-E1)
- R27 pad 2: Net-(C3-Pad2) -> Net-(R27-Pad2)
- R32 pad 1: Net-(U4B-+) -> Net-(U4B--)
- R33 pad 1: Net-(U5A-E) -> Net-(U5A-E1)
- R33 pad 2: Net-(C14-Pad2) -> Net-(R33-Pad2)
- R9 pad 2: Net-(U3C--) -> Net-(R24-Pad1)
- RV5 pad 2: Net-(U2A-B) -> Net-(U2A-B1)
- RV6 pad 2: Net-(U5A-B) -> Net-(U5A-B1)
- U1 pad 12: Net-(U1D-+) -> GND
- U1 pad 13: GND -> Net-(U1D--)
- U2 pad 1: Net-(U2A-B) -> Net-(U2A-E1)
- U2 pad 2: GND -> Net-(U2A-B1)
- U2 pad 4: Net-(U2A-E) -> Net-(U2A-E1)
- U2 pad 5: Net-(U2A-E) -> GND
- U2 pad 6: Net-(U1D-+) -> Net-(U1D--)
- U4 pad 5: Net-(U4B-+) -> GND
- U4 pad 6: GND -> Net-(U4B--)
- U5 pad 1: Net-(U5A-B) -> Net-(U5A-E1)
- U5 pad 2: GND -> Net-(U5A-B1)
- U5 pad 4: Net-(U5A-E) -> Net-(U5A-E1)
- U5 pad 5: Net-(U5A-E) -> GND
- U5 pad 6: Net-(U4B-+) -> Net-(U4B--)
Routing:
- net CV_A: track 72.4 -> 0.00 mm
- net Net-(C14-Pad2): track 8.06 -> 59.1 mm, vias 0 -> 2
- net Net-(R33-Pad2): track 0.00 -> 51.0 mm, vias 0 -> 1
- net Net-(U5A-B1): track 0.00 -> 46.9 mm, vias 0 -> 1
- net Net-(U5B-C2): track 68.2 -> 23.1 mm
- net +12V: track 137.6 -> 92.9 mm
- net -12V: track 124.4 -> 86.9 mm, vias 7 -> 3
- net Net-(U4A--): track 49.4 -> 14.3 mm
- net Net-(R22-Pad1): track 23.3 -> 57.6 mm, vias 0 -> 2
- net Net-(R29-Pad2): track 10.9 -> 42.4 mm, vias 0 -> 1
- net Net-(J10-Pin_5): track 4.79 -> 33.4 mm, vias 0 -> 2
- net Net-(C3-Pad2): track 8.97 -> 36.9 mm, vias 0 -> 2
- net Net-(R27-Pad2): track 0.00 -> 26.9 mm
- net Net-(R19-Pad2): track 4.34 -> 27.4 mm, vias 0 -> 1
- net Net-(U3A--): track 32.4 -> 9.35 mm, vias 2 -> 0
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Other:
- board text added: "1. Input at 10V p2p 2. Set CV at 5V 3. Trim SHAPE until output at 10V p2p (unity gain) 4. Set CV at 1V 5. Trim SLOPE until output at 625mV 6. Repeat from step 2 7. Set CV at 6V 8. Use TRIM to cap gain slightly above unity"
- board text added: "SHAPE"
- board text added: "SLOPE"
- board text added: "TRIM"
- board text added: "VCA-2 Exp ver. 1.1 BC857BS 3/2026"
