File: exp-vintage-vca/exp-vintage-vca.kicad_sch (KiCad schematic)
At the start: 81 parts, among them J1 AudioJack2, J10 Conn_01x10_Socket, J11 Conn_01x04_Pin, J12 Conn_01x04_Socket, J13 AudioJack2, J14 AudioJack2, J15 Conn_02x08_Odd_Even, J2 AudioJack2, J3 AudioJack2, J4 AudioJack2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

Commit message: Exponential VCA ver. 1.2
Parts:
- removed JP1: SolderJumper_2_Open, Jumper:SolderJumper-2_P1.3mm_Open_RoundedPad1.0x1.5mm, symbol Jumper:SolderJumper_2_Open
- removed TP1, TP2, TP3, TP4: TestPoint, TestPoint:TestPoint_Loop_D1.80mm_Drill1.0mm_Beaded, symbol Connector:TestPoint
- removed U5: ~, Package_TO_SOT_SMD:SOT-363_SC-70-6, symbol linear_vintage_vca:pmp5201
- added D3, D5: SS14, Diode_SMD:D_SMA, symbol Diode:SS14
- added FB1, FB2: FerriteBead_Small, linear_vintage_vca:Ferrite_Bead_5mm_3.5mm_Horizontal, symbol Device:FerriteBead_Small
- added R24, R35: 10K, Resistor_SMD:R_0603_1608Metric_Pad0.98x0.95mm_HandSolder, symbol Device:R
- added RV10: 20K, Potentiometer_THT:Potentiometer_Bourns_3296W_Vertical, symbol Device:R_Potentiometer_Trim
- added RV9: 20k, Potentiometer_THT:Potentiometer_Bourns_3296W_Vertical, symbol Device:R_Potentiometer_Trim
- added U5: BC857BS, Package_TO_SOT_SMD:SOT-363_SC-70-6, symbol Transistor_BJT:BC857BS
- C1, C2: LCSC (none) -> C46653
- C10, C13, C4, C5, C6, C7, C8, C9: LCSC (none) -> C49678
- C11, C12: footprint Capacitor_THT:CP_Radial_D10.0mm_P2.50mm_P5.00mm -> Capacitor_THT:CP_Radial_D5.0mm_P2.50mm; LCSC (none) -> C13585; now left out of the parts list
- C14, C3: LCSC (none) -> C1790
- D1, D2: footprint Diode_SMD:D_0805_2012Metric_Pad1.15x1.40mm_HandSolder -> Diode_SMD:D_SOD-123; LCSC (none) -> C81598
- J10, J12, J9: now left out of the parts list
- J15: footprint Connector_IDC:IDC-Header_2x08_P2.54mm_Vertical -> Connector_IDC:IDC-Header_2x05_P2.54mm_Vertical; symbol Connector_Generic:Conn_02x08_Odd_Even -> Connector_Generic:Conn_02x05_Odd_Even
- R10, R9: footprint Resistor_SMD:R_0805_2012Metric_Pad1.20x1.40mm_HandSolder -> Resistor_SMD:R_0603_1608Metric_Pad0.98x0.95mm_HandSolder; LCSC (none) -> C25803
- R11, R12, R15, R16: value 620R -> 680R; footprint Resistor_SMD:R_0805_2012Metric_Pad1.20x1.40mm_HandSolder -> Resistor_SMD:R_0603_1608Metric_Pad0.98x0.95mm_HandSolder; LCSC (none) -> C23228
- R13, R14: footprint Resistor_SMD:R_0805_2012Metric_Pad1.20x1.40mm_HandSolder -> Resistor_SMD:R_0603_1608Metric_Pad0.98x0.95mm_HandSolder; LCSC (none) -> C4216
- R17, R23: value 330k -> 330K; footprint Resistor_SMD:R_0805_2012Metric_Pad1.20x1.40mm_HandSolder -> Resistor_SMD:R_0603_1608Metric_Pad0.98x0.95mm_HandSolder; LCSC (none) -> C23137
- R18, R29, R3, R4, R5, R6, R7, R8: footprint Resistor_SMD:R_0805_2012Metric_Pad1.20x1.40mm_HandSolder -> Resistor_SMD:R_0603_1608Metric_Pad0.98x0.95mm_HandSolder; LCSC (none) -> C23137
- R19, R20: value 20k -> 10K; footprint Resistor_SMD:R_0805_2012Metric_Pad1.20x1.40mm_HandSolder -> Resistor_SMD:R_0603_1608Metric_Pad0.98x0.95mm_HandSolder; LCSC (none) -> C4184
- R21, R22: footprint Resistor_SMD:R_0805_2012Metric_Pad1.20x1.40mm_HandSolder -> Resistor_SMD:R_0603_1608Metric_Pad0.98x0.95mm_HandSolder; LCSC (none) -> C21190
- R25, R31: value 330 -> 10; footprint Resistor_SMD:R_0805_2012Metric_Pad1.20x1.40mm_HandSolder -> Resistor_SMD:R_0603_1608Metric_Pad0.98x0.95mm_HandSolder; LCSC (none) -> C23138
- R26, R32: value 1Meg -> 2Meg; footprint Resistor_SMD:R_0805_2012Metric_Pad1.20x1.40mm_HandSolder -> Resistor_SMD:R_0603_1608Metric_Pad0.98x0.95mm_HandSolder; LCSC (none) -> C22935
- R27, R33: value 22k -> 10K; footprint Resistor_SMD:R_0805_2012Metric_Pad1.20x1.40mm_HandSolder -> Resistor_SMD:R_0603_1608Metric_Pad0.98x0.95mm_HandSolder; LCSC (none) -> C31850
- R28, R34: value 6k8 -> 20K; footprint Resistor_SMD:R_0805_2012Metric_Pad1.20x1.40mm_HandSolder -> Resistor_SMD:R_0603_1608Metric_Pad0.98x0.95mm_HandSolder; LCSC (none) -> C23212
- RV5, RV6: footprint Potentiometer_THT:Potentiometer_Runtron_RM-065_Vertical -> Potentiometer_THT:Potentiometer_Bourns_3296W_Vertical; now left out of the parts list
- RV7, RV8: value 10k -> 20K; footprint Potentiometer_THT:Potentiometer_Runtron_RM-065_Vertical -> Potentiometer_THT:Potentiometer_Bourns_3296W_Vertical; now left out of the parts list
- U1: footprint Package_SO:SOIC-14_3.9x8.7mm_P1.27mm -> linear_vintage_vca:SOT-23-THIN-14_2x4.2mm_P0.5mm; symbol Amplifier_Operational:TL074 -> linear_vintage_vca:TL074; LCSC (none) -> C5116353; Rotation Offset (none) -> 90
- U2: value ~ -> BC857BS; symbol linear_vintage_vca:pmp5201 -> Transistor_BJT:BC857BS; LCSC (none) -> C8654; Rotation Offset (none) -> 90
- U3: symbol Amplifier_Operational:LM13700 -> linear_vintage_vca:LM13700; LCSC (none) -> C174050
- U4: footprint Package_SO:SOIC-14_3.9x8.7mm_P1.27mm -> linear_vintage_vca:SOT-23-THIN-14_2x4.2mm_P0.5mm; symbol Amplifier_Operational:TL074 -> linear_vintage_vca:TL074; LCSC (none) -> C5116353
Connections:
- net CV_A is gone; now on net GND_A: J1.TN, J11.1 (Pin_1), J3.TN
- net +12V: now also FB1.1; no longer J15.10 (Pin_10), J15.9 (Pin_9)
- net -12V: now also FB2.1; no longer J15.1 (Pin_1), J15.2 (Pin_2)
- net GND: now also J12.1 (Pin_1), U1.12 (+), U2.5 (B2), U4.5 (+), U5.5 (B2); no longer U1.13 (-), U2.2 (B), U4.6 (-)
- net at R12.1, U3.13 (-): now also R35.2; no longer R10.2
- net at R27.1, U2.4 (E2): now also U2.1 (E1); no longer U2.5 (E)
- net at C3.2, U1.14: now also RV9.2, RV9.3; no longer R27.2
- net at R33.1: now also U5.1 (E1), U5.4 (E2)
- net at C14.2, U4.7: now also RV10.2, RV10.3; no longer R33.2
- net at R11.1, U3.4 (-): now also R24.2; no longer R9.2
- net at C14.1, R32.1: now also U4.6 (-), U5.6 (C1); no longer U4.5 (+)
- net at C3.1, R26.1, U2.6 (C1): now also U1.13 (-); no longer U1.12 (+)
- net at R34.1: now also U5.3 (C2)
- net at RV5.2: now also U2.2 (B1); no longer U2.1 (B)
- net at RV6.2: now also U5.2 (B1)
- removed net +5V: J15.11 (Pin_11), J15.12 (Pin_12)
- removed net CV_B: J15.13 (Pin_13), J15.14 (Pin_14)
- new net: R33.2, RV10.1
- new net: R10.2, R35.1
- new net: R27.2, RV9.1
- new net: D3.1 (K), FB1.2
- new net: D3.2 (A), J15.10 (Pin_10), J15.9 (Pin_9)
- new net: R24.1, R9.2
- new net: D5.1 (K), J15.1 (Pin_1), J15.2 (Pin_2)
- new net: D5.2 (A), FB2.2
- no-connect marks 0 -> 2
Other:
- moved on the sheet: C14, C3, R10, R11, R12, R15, R16, R32, R9, U1D, U4B
