File: simulations/antialiasing-input-stage/antialiasing-input-stage.kicad_sch (KiCad schematic)
At the start: 13 parts, among them U1 MCP6002

Commit message: Update input stage for +/-10V (20Vpp) input signal and regenerate simulation
Co-authored-by: stash-s <6302220+stash-s@users.noreply.github.com>
Parts:
- C1: value 330p -> 680p
- C2: value 180p -> 360p
- R2: value 30.1k -> 15k
- R_PD: value 150k -> 43.2k
- R_PU: value 60.4k -> 30.1k
- V1: value SIN(0 5 1k) -> SIN(0 10 1k)
Changed lines of the file:
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@@
 		(in_bom yes) (on_board yes)
 		(property "Reference" "V1" (at 33.02 111.76 0) (effects (font (size 1.27 1.27))))
-		(property "Value" "SIN(0 5 1k)" (at 33.02 114.3 0) (effects (font (size 1.27 1.27))))
-		(property "Sim.Params" "dc=0 ampl=5 f=1k ac=1" (at 25.4 114.3 0) (effects (font (size 1.27 1.27)) (hide yes)))
+		(property "Value" "SIN(0 10 1k)" (at 33.02 114.3 0) (effects (font (size 1.27 1.27))))
+		(property "Sim.Params" "dc=0 ampl=10 f=1k ac=1" (at 25.4 114.3 0) (effects (font (size 1.27 1.27)) (hide yes)))
 		(pin "1")
 		(pin "2")
@@
 		(in_bom yes) (on_board yes)
 		(property "Reference" "R_PU" (at 64.77 62.23 0) (effects (font (size 1.27 1.27))))
-		(property "Value" "60.4k" (at 64.77 64.77 0) (effects (font (size 1.27 1.27))))
+		(property "Value" "30.1k" (at 64.77 64.77 0) (effects (font (size 1.27 1.27))))
 		(pin "1")
 		(pin "2")
@@
 		(in_bom yes) (on_board yes)
 		(property "Reference" "R_PD" (at 64.77 87.63 0) (effects (font (size 1.27 1.27))))
-		(property "Value" "150k" (at 64.77 90.17 0) (effects (font (size 1.27 1.27))))
+		(property "Value" "43.2k" (at 64.77 90.17 0) (effects (font (size 1.27 1.27))))
 		(pin "1")
 		(pin "2")
@@
 		(in_bom yes) (on_board yes)
 		(property "Reference" "R2" (at 81.28 72.39 0) (effects (font (size 1.27 1.27))))
-		(property "Value" "30.1k" (at 81.28 80.01 0) (effects (font (size 1.27 1.27))))
+		(property "Value" "15k" (at 81.28 80.01 0) (effects (font (size 1.27 1.27))))
 		(pin "1")
 		(pin "2")
@@
 		(in_bom yes) (on_board yes)
 		(property "Reference" "C2" (at 97.79 87.63 0) (effects (font (size 1.27 1.27))))
-		(property "Value" "180p" (at 97.79 90.17 0) (effects (font (size 1.27 1.27))))
+		(property "Value" "360p" (at 97.79 90.17 0) (effects (font (size 1.27 1.27))))
 		(pin "1")
 		(pin "2")
@@
 		(in_bom yes) (on_board yes)
 		(property "Reference" "C1" (at 101.6 46.99 0) (effects (font (size 1.27 1.27))))
-		(property "Value" "330p" (at 101.6 54.61 0) (effects (font (size 1.27 1.27))))
+		(property "Value" "680p" (at 101.6 54.61 0) (effects (font (size 1.27 1.27))))
 		(pin "1")
 		(pin "2")

Commit message: Use E12 resistor and E6 capacitor standard series values
Co-authored-by: stash-s <6302220+stash-s@users.noreply.github.com>
Parts:
- C2: value 360p -> 330p
- R2: value 15k -> 18k
- R_PD: value 43.2k -> 39k
- R_PU: value 30.1k -> 27k
Changed lines of the file:
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@@
 		(in_bom yes) (on_board yes)
 		(property "Reference" "R_PU" (at 64.77 62.23 0) (effects (font (size 1.27 1.27))))
-		(property "Value" "30.1k" (at 64.77 64.77 0) (effects (font (size 1.27 1.27))))
+		(property "Value" "27k" (at 64.77 64.77 0) (effects (font (size 1.27 1.27))))
 		(pin "1")
 		(pin "2")
@@
 		(in_bom yes) (on_board yes)
 		(property "Reference" "R_PD" (at 64.77 87.63 0) (effects (font (size 1.27 1.27))))
-		(property "Value" "43.2k" (at 64.77 90.17 0) (effects (font (size 1.27 1.27))))
+		(property "Value" "39k" (at 64.77 90.17 0) (effects (font (size 1.27 1.27))))
 		(pin "1")
 		(pin "2")
@@
 		(in_bom yes) (on_board yes)
 		(property "Reference" "R2" (at 81.28 72.39 0) (effects (font (size 1.27 1.27))))
-		(property "Value" "15k" (at 81.28 80.01 0) (effects (font (size 1.27 1.27))))
+		(property "Value" "18k" (at 81.28 80.01 0) (effects (font (size 1.27 1.27))))
 		(pin "1")
 		(pin "2")
@@
 		(in_bom yes) (on_board yes)
 		(property "Reference" "C2" (at 97.79 87.63 0) (effects (font (size 1.27 1.27))))
-		(property "Value" "360p" (at 97.79 90.17 0) (effects (font (size 1.27 1.27))))
+		(property "Value" "330p" (at 97.79 90.17 0) (effects (font (size 1.27 1.27))))
 		(pin "1")
 		(pin "2")

Commit message: Kicad  v10 schematic for antialiasing input stage
Parts:
- removed D1, D2: BAT54, symbol Device:D
- removed U1: MCP6002, symbol Simulation_SPICE:OPAMP
- added D3, D4: D, symbol Simulation_SPICE:D
- added U2: ${SIM.PARAMS}, Package_SO:SO-20-1EP_7.52x12.825mm_P1.27mm_EP6.045x12.09mm_Mask3.56x4.47mm, symbol Simulation_SPICE:OPAMP
- V1: value SIN(0 10 1k) -> VSIN; footprint (none) -> Package_QFP:TQFP-44_10x10mm_P0.8mm
- renumbered C2 to C1, C1 to C2, C_ADC to C_ADC1, R_ADC to R_ADC1, R_PD to R_PD1, R_PU to R_PU1
Connections:
- net +3.3V: now also D3.1 (K), U2.3 (V+); no longer C2.1, R1.2, R2.1, R_PD1.1, R_PU1.2
- net GND: now also D4.2 (A), U2.4 (V-)
- net OUT: now also U2.2 (-), U2.5
- net N_INP: now reaches C1.1, R2.2
- net N_INP: now also U2.1 (+)
- new net N1: C2.1, D3.2 (A), D4.1 (K), R1.2, R2.1, R_PD1.1, R_PU1.2

Commit message: Smoothen the kicad schematic.
Parts:
- removed V2: 3.3V, symbol Simulation_SPICE:VDC
- added V3: 1, symbol Simulation_SPICE:VDC
Connections:
- net +3.3V: now also V3.1
- net GND: now also V3.2
Other:
- moved on the sheet: C1, C2, D3, D4, R1, R2, R_ADC1, R_PD1, R_PU1, U2
